Commit message: add namespace in robot_description

File: qupa_description/urdf/bases/base.xacro (robot description, xacro)
@@ -10,5 +10,5 @@
             <origin xyz="0.0 0.0 -0.0" rpy="0 0 0"/>
         </joint> -->
-        <link name="base_link">
+        <link name="$(arg tf_prefix)/base_link">
             <inertial>
                 <origin xyz="0 0 0" rpy="0 0 0" />
@@ -37,9 +37,9 @@
         </link>
         <joint name="imu_joint" type="fixed">
-            <parent link="base_link"/>
-            <child link="imu_link"/>
+            <parent link="$(arg tf_prefix)/base_link"/>
+            <child link="$(arg tf_prefix)/imu_link"/>
             <origin xyz="0.0 0 0.07" rpy="0 0 0"/>
         </joint>
-        <link name="imu_link">
+        <link name="$(arg tf_prefix)/imu_link">
             <inertial>
                 <mass value="0.05"/>

File: qupa_description/urdf/bases/module.xacro (robot description, xacro)
@@ -5,5 +5,5 @@
     <!--Base with Module installed-->
     <xacro:macro name="module">
-        <link name="base_link">
+        <link name="$(arg tf_prefix)/base_link">
             <inertial>
                 <origin xyz="0 0 0" rpy="0 0 0" />
@@ -32,9 +32,9 @@
         </link>
         <joint name="imu_joint" type="fixed">
-            <parent link="base_link"/>
-            <child link="imu_link"/>
+            <parent link="$(arg tf_prefix)/base_link"/>
+            <child link="$(arg tf_prefix)/imu_link"/>
             <origin xyz="0.0 0 0.07" rpy="0 0 0"/>
         </joint>
-        <link name="imu_link">
+        <link name="$(arg tf_prefix)/imu_link">
             <inertial>
                 <mass value="0.05"/>

File: qupa_description/urdf/gazebo_plugins.xacro (robot description, xacro)
@@ -30,5 +30,5 @@
         </plugin>
     </gazebo>
-    <gazebo reference="imu_link">
+    <gazebo reference="$(arg tf_prefix)/imu_link">
         <gravity>true</gravity>
         <sensor name="imu_sensor" type="imu">
@@ -39,10 +39,10 @@
         <plugin filename="libgazebo_ros_imu_sensor.so" name="$(arg tf_prefix)_imu_plugin">
             <topicName>$(arg tf_prefix)/imu</topicName>
-            <bodyName>imu_link</bodyName>
+            <bodyName>$(arg tf_prefix)/imu_link</bodyName>
             <updateRateHZ>10.0</updateRateHZ>
             <gaussianNoise>0.0</gaussianNoise>
             <xyzOffset>0 0 0</xyzOffset>
             <rpyOffset>0 0 0</rpyOffset>
-            <frameName>imu_link</frameName>
+            <frameName>$(arg tf_prefix)/imu_link</frameName>
             <initialOrientationAsReference>false</initialOrientationAsReference>
         </plugin>

File: qupa_description/urdf/qupa.xacro (robot description, xacro)
@@ -2,5 +2,5 @@
 <robot xmlns:xacro="http://www.ros.org/wiki/xacro" name="$(arg tf_prefix)">
     <xacro:property name="M_PI" value="3.1415926535897931" />
-    <xacro:property name="tf_prefix" default="qp_1"/>
+    <xacro:property name="tf_prefix" value="$(arg tf_prefix)"/>
     <xacro:property name="high_res" value="$(arg high_res)" lazy_eval="false"/>
     <xacro:property name="module" value="$(arg module)" lazy_eval="false"/>
@@ -33,10 +33,10 @@
         <xacro:link_1
             prefix="Left"
-            parent_link="base_link"
+            parent_link="${tf_prefix}/base_link"
             xyz="0.042536 0.012084 0.0782"
             rpy="0 0 0.55"/>
         <xacro:link_1
             prefix="Right"
-            parent_link="base_link"
+            parent_link="${tf_prefix}/base_link"
             xyz="0.042536 -0.012116 0.0782"
             rpy="0 0 -0.43481"/>
@@ -78,25 +78,25 @@
     <!-- Wheels Macro-->
     <xacro:wheel
-        wheel_name="R_wheel"
+        wheel_name="${tf_prefix}/R_wheel"
         wheel_joint_name="R_wheel_joint"
-        wheel_parent_name="base_link"
+        wheel_parent_name="${tf_prefix}/base_link"
         wheel_joint_origin_xyz="-0 0.0415 0.016"
         wheel_joint_origin_rpy=" 1.5708 0 3.1416" />
     <xacro:wheel
-        wheel_name="L_wheel"
+        wheel_name="${tf_prefix}/L_wheel"
         wheel_joint_name="L_wheel_joint"
-        wheel_parent_name="base_link"
+        wheel_parent_name="${tf_prefix}/base_link"
         wheel_joint_origin_xyz="0 -0.0415 0.016"
         wheel_joint_origin_rpy=" 1.5708 0 0" />
     <xacro:caster
-        link_name = "caster_R"
+        link_name = "${tf_prefix}/caster_R"
         joint_name = "caster_R_joint"
         joint_origin_xyz = "0.0305 -0.0265 0.005"/>
     <xacro:caster
-        link_name = "caster_L"
+        link_name = "${tf_prefix}/caster_L"
         joint_name = "caster_L_joint"
         joint_origin_xyz = "0.0305 0.0265 0.005"/>
     <xacro:caster
-        link_name = "caster_B"
+        link_name = "${tf_prefix}/caster_B"
         joint_name = "caster_B_joint"
         joint_origin_xyz = "-0.0325 0 0.005"/>

File: qupa_description/urdf/sensors/color.xacro (robot description, xacro)
@@ -2,5 +2,5 @@
 <robot xmlns:xacro="http://www.ros.org/wiki/xacro" name="$(arg tf_prefix)">
   <xacro:macro name="color_camera">
-    <link name="color_camera_link">
+    <link name="$(arg tf_prefix)/color_camera_link">
       <!-- <inertial>
         <origin
@@ -46,7 +46,7 @@
         rpy="0 0 0" />
       <parent
-        link="base_link" />
+        link="$(arg tf_prefix)/base_link" />
       <child
-        link="color_camera_link" />
+        link="$(arg tf_prefix)/color_camera_link" />
       <axis
         xyz="0 0 1" />

File: qupa_description/urdf/sensors/infrared.xacro (robot description, xacro)
@@ -7,5 +7,5 @@
                                         joint_origin_xyz joint_origin_rpy">
     <!--Link Definition -->
-    <link name="${link_name}">
+    <link name="$(arg tf_prefix)/${link_name}">
       <inertial>
         <mass value="0.01"/>
@@ -25,6 +25,6 @@
     <joint name="${joint_name}" type="fixed">
       <origin xyz="${joint_origin_xyz}" rpy="${joint_origin_rpy}" />
-      <parent link="base_link" />
-      <child link="${link_name}" />
+      <parent link="$(arg tf_prefix)/base_link" />
+      <child link="$(arg tf_prefix)/${link_name}" />
       <axis xyz="0 0 0" />
     </joint>
@@ -33,5 +33,5 @@
   <xacro:macro name="infrared" params="joint_origin_xyz joint_origin_rpy">
     <!--Link Definition -->
-    <link name="infrared_link">
+    <link name="$(arg tf_prefix)/infrared_link">
       <inertial>
         <mass value="0.0001"/>
@@ -55,6 +55,6 @@
     <joint name="infrared_joint" type="fixed">
       <origin xyz="${joint_origin_xyz}" rpy="${joint_origin_rpy}" />
-      <parent link="base_link" />
-      <child link="infrared_link" />
+      <parent link="$(arg tf_prefix)/base_link" />
+      <child link="$(arg tf_prefix)/infrared_link" />
       <axis xyz="0 0 0" />
     </joint>

File: qupa_description/urdf/sensors/mirror.xacro (robot description, xacro)
@@ -6,5 +6,5 @@
     <!-- Mirror Macro -->
     <xacro:macro name="mirror">
-        <link name="mirror_link">
+        <link name="$(arg tf_prefix)/mirror_link">
             <inertial>
             <origin
@@ -38,6 +38,6 @@
         <joint name="mirror_joint" type="fixed">
             <origin xyz="0 0 ${mirror_height}" rpy="1.5708 0 0" />
-            <parent link="base_link" />
-            <child link="mirror_link" />
+            <parent link="$(arg tf_prefix)/base_link" />
+            <child link="$(arg tf_prefix)/mirror_link" />
             <axis xyz="1 0 0" />
         </joint>
@@ -46,5 +46,5 @@
     <xacro:macro name="log_cam">
         <!--Logical Camera Frame-->
-        <link name="logical_camera_link">
+        <link name="$(arg tf_prefix)/logical_camera_link">
             <inertial>
                 <mass value="0.001" />
@@ -61,6 +61,6 @@
         <!--Logical Camera joint-->
         <joint name="logical_camera_joint" type="fixed">
-            <parent link="base_link" />
-            <child link="logical_camera_link" />
+            <parent link="$(arg tf_prefix)/base_link" />
+            <child link="$(arg tf_prefix)/logical_camera_link" />
             <origin xyz="0 0 ${camera_height}"  rpy="0 1.5708 0" />
         </joint>
@@ -82,5 +82,5 @@
     <xacro:macro name="real_cam">
         <!--Logical Camera Frame-->
-        <link name="camera_link">
+        <link name="$(arg tf_prefix)/camera_link">
             <inertial>
                 <mass value="0.001" />
@@ -97,6 +97,6 @@
         <!--Logical Camera joint-->
         <joint name="camera_joint" type="fixed">
-            <parent link="base_link" />
-            <child link="camera_link" />
+            <parent link="$(arg tf_prefix)/base_link" />
+            <child link="$(arg tf_prefix)/camera_link" />
             <origin xyz="0 0 ${camera_height}"  rpy="0 1.5708 0" />
         </joint>

File: qupa_description/urdf/wheels/caster.xacro (robot description, xacro)
@@ -30,5 +30,5 @@
     <joint name="${joint_name}" type="fixed">
       <origin xyz="${joint_origin_xyz}" rpy="0 0 0" />
-      <parent link="base_link" />
+      <parent link="$(arg tf_prefix)/base_link" />
       <child link="${link_name}" />
     </joint>
