Commit message: add urdf descriptions for leds sim plugin and stl meshes

File: qupa_description/urdf/bases/base.xacro (robot description, xacro)
@@ -3,4 +3,14 @@
     <xacro:property name="base_mass" value="1" />
     <xacro:property name="base_scale" value="1 1 1" />
+    <!-- Real robot is white -->
+    <material name="white">
+        <color rgba="0.9 0.9 0.9 1.0" />
+    </material>
+    <!-- Acrylic dome: WHITE translucent diffuser the LEDs glow through.
+         acrylic_alpha: 0 = invisible, 1 = fully opaque. Lower = lighter/clearer. -->
+    <xacro:property name="acrylic_alpha" value="0.90" />
+    <material name="acrylic">
+        <color rgba="1.0 1.0 1.0 ${acrylic_alpha}" />
+    </material>
     <xacro:macro name="base">
         <!-- <link name="base_footprint"/>
@@ -22,18 +32,51 @@
                     izz="0.00180" />
                 </inertial>
-            <visual>
+            <!-- Body shell (opaque). The acrylic dome lives on its OWN link
+                 (acrylic_dome_link, below) so led_sim_node can drive its
+                 emissive colour by a clean, stable visual name. -->
+            <visual name="base_body">
                 <origin xyz="0 0 0" rpy="0 0 0" />
                 <geometry>
-                    <mesh filename="package://qupa_description/meshes/qupa.dae" scale="${base_scale}" />
+                    <mesh filename="package://qupa_description/meshes/base.stl" scale="${base_scale}" />
                 </geometry>
+                <material name="white" />
             </visual>
             <collision>
                 <origin xyz="0 0 0" rpy="0 0 0" />
                 <geometry>
-                    <mesh filename="package://qupa_description/meshes/qupa.dae" scale="${base_scale}" />
+                    <mesh filename="package://qupa_description/meshes/base.stl" scale="${base_scale}" />
                 </geometry>
                 <self_collide>false</self_collide>
             </collision>
         </link>
+        <!-- ── Acrylic dome — own link so its visual has a clean, stable name
+             (qupa/acrylic_dome_link_visual) that led_sim_node targets via
+             material_color to make the dome GLOW in the LED colour (the
+             "difuminado" look).  Nameless visual + disableFixedJointLumping →
+             sdformat auto-names it <link>_visual.  Visual only. -->
+        <link name="$(arg tf_prefix)/acrylic_dome_link">
+            <inertial>
+                <mass value="1e-5" />
+                <origin xyz="0 0 0" rpy="0 0 0" />
+                <inertia ixx="1e-9" ixy="0" ixz="0"
+                         iyy="1e-9" iyz="0" izz="1e-9" />
+            </inertial>
+            <visual>
+                <origin xyz="0 0 0" rpy="0 0 0" />
+                <geometry>
+                    <mesh filename="package://qupa_description/meshes/dome.stl" scale="${base_scale}" />
+                </geometry>
+                <material name="acrylic" />
+            </visual>
+        </link>
+        <joint name="acrylic_dome_joint" type="fixed">
+            <parent link="$(arg tf_prefix)/base_link" />
+            <child  link="$(arg tf_prefix)/acrylic_dome_link" />
+            <origin xyz="0 0 0" rpy="0 0 0" />
+        </joint>
+        <gazebo reference="acrylic_dome_joint">
+            <disableFixedJointLumping>true</disableFixedJointLumping>
+            <preserveFixedJoint>true</preserveFixedJoint>
+        </gazebo>
         <joint name="imu_joint" type="fixed">
             <parent link="$(arg tf_prefix)/base_link"/>

File: qupa_description/urdf/gazebo_plugins.xacro (robot description, xacro)
@@ -1,52 +1,38 @@
 <robot xmlns:xacro="http://www.ros.org/wiki/xacro" name="$(arg tf_prefix)">
+  <!--
+    gazebo_plugins.xacro
+    Gazebo Harmonic (gz-sim) plugin definitions for the QUPA robot.
+    Only included when use_sim_plugins:=true (i.e. when spawning in Gazebo).
+    Desktop / hardware launches should keep use_sim_plugins:=false.
+  -->
+  <xacro:if value="${use_sim_plugins}">
+    <!-- ───────────────────────────────────────────────────────────────
+         DIFFERENTIAL DRIVE  (gz::sim::systems::DiffDrive)
+         Publishes:  /{tf_prefix}/odom   (gz topic → ros_gz_bridge)
+                     /tf                 (gz topic → ros_gz_bridge)
+         Subscribes: /{tf_prefix}/cmd_vel (ros_gz_bridge → gz topic)
+    ─────────────────────────────────────────────────────────────────── -->
     <gazebo>
-        <plugin name="$(arg tf_prefix)_diff_drive_controller" filename="libgazebo_ros_diff_drive.so">
-            <ros>
-                <namespace>$(arg tf_prefix)</namespace>
-                <remapping>
-                    <remap from="cmd_vel" to="$(arg tf_prefix)/cmd_vel" />
-                    <remap from="odom" to="$(arg tf_prefix)/odom" />
-                </remapping>
-            </ros>
-            <legacyMode>true</legacyMode>
-            <!-- <robotNamespace>$(arg tf_prefix)</robotNamespace> -->
-            <updateRate>40.0</updateRate>
-            <leftJoint>L_wheel_joint</leftJoint>
-            <rightJoint>R_wheel_joint</rightJoint>
-            <wheelSeparation>0.088</wheelSeparation>
-            <wheelDiameter>0.032</wheelDiameter>
-            <wheelAcceleration> 0.1</wheelAcceleration>
-            <wheelTorque>15</wheelTorque>
-            <rosDebugLevel>na</rosDebugLevel>
-            <robotBaseFrame>$(arg tf_prefix)/base_link</robotBaseFrame>
-            <commandTopic>$(arg tf_prefix)/cmd_vel</commandTopic>
-            <odometryTopic>$(arg tf_prefix)/odom</odometryTopic>
-            <odometryFrame>$(arg tf_prefix)/odom</odometryFrame>
-            <publishWheelTF>true</publishWheelTF>
-            <publishOdomTF>true</publishOdomTF>
-            <publishWheelJointState>false</publishWheelJointState>
-            <publishTf>1</publishTf>
-            <odometrySource>world</odometrySource>
-        </plugin>
+      <plugin filename="gz-sim-diff-drive-system"
+              name="gz::sim::systems::DiffDrive">
+        <left_joint>L_wheel_joint</left_joint>
+        <right_joint>R_wheel_joint</right_joint>
+        <wheel_separation>0.088</wheel_separation>
+        <wheel_radius>0.016</wheel_radius>
+        <!-- velocity / acceleration limits matching the real robot -->
+        <max_velocity>0.08</max_velocity>
+        <max_angular_velocity>2.5</max_angular_velocity>
+        <max_linear_acceleration>0.1</max_linear_acceleration>
+        <max_angular_acceleration>10.0</max_angular_acceleration>
+        <!-- gz-transport topic names (bridged to ROS by ros_gz_bridge) -->
+        <topic>/$(arg tf_prefix)/cmd_vel</topic>
+        <odom_topic>/$(arg tf_prefix)/odom</odom_topic>
+        <tf_topic>/tf</tf_topic>
+        <!-- TF frame names -->
+        <frame_id>$(arg tf_prefix)/odom</frame_id>
+        <child_frame_id>$(arg tf_prefix)/base_link</child_frame_id>
+        <odom_publish_frequency>40</odom_publish_frequency>
+      </plugin>
     </gazebo>
-    <gazebo reference="$(arg tf_prefix)/imu_link">
-        <gravity>true</gravity>
-        <sensor name="imu_sensor" type="imu">
-        <always_on>true</always_on>
-        <update_rate>100</update_rate>
-        <visualize>true</visualize>
-        <topic>__default_topic__</topic>
-        <plugin filename="libgazebo_ros_imu_sensor.so" name="$(arg tf_prefix)_imu_plugin">
-            <topicName>$(arg tf_prefix)/imu</topicName>
-            <bodyName>$(arg tf_prefix)/imu_link</bodyName>
-            <updateRateHZ>10.0</updateRateHZ>
-            <gaussianNoise>0.0</gaussianNoise>
-            <xyzOffset>0 0 0</xyzOffset>
-            <rpyOffset>0 0 0</rpyOffset>
-            <frameName>$(arg tf_prefix)/imu_link</frameName>
-            <initialOrientationAsReference>false</initialOrientationAsReference>
-        </plugin>
-        <pose>0 0 0 0 0 0</pose>
-        </sensor>
-    </gazebo>
+  </xacro:if>
 </robot>

File: qupa_description/urdf/qupa.xacro (robot description, xacro)
@@ -2,9 +2,13 @@
 <robot xmlns:xacro="http://www.ros.org/wiki/xacro" name="$(arg tf_prefix)">
     <xacro:property name="M_PI" value="3.1415926535897931" />
-    <xacro:property name="tf_prefix" value="$(arg tf_prefix)"/>
-    <xacro:property name="high_res" value="$(arg high_res)" lazy_eval="false"/>
-    <xacro:property name="module" value="$(arg module)" lazy_eval="false"/>
+    <xacro:property name="tf_prefix"       value="$(arg tf_prefix)"/>
+    <xacro:property name="high_res"        value="$(arg high_res)"        lazy_eval="false"/>
+    <xacro:property name="module"          value="$(arg module)"          lazy_eval="false"/>
+    <xacro:property name="use_sim_plugins" value="$(arg use_sim_plugins)" lazy_eval="false"/>
     <xacro:property name="base_height" value="0.0" />
     <xacro:property name="mirror_height" value="${base_height + 0.2}" />
+    <!-- IR ring inset: <1 pulls the IR sensors radially INWARD (more recessed
+         into the body). 1.0 = original edge position; 0.82 ≈ 1 cm inward. -->
+    <xacro:property name="ir_inset_scale" value="0.82" />
     <!--Include Xacro files -->
     <xacro:include filename="$(find qupa_description)/urdf/wheels/wheel.xacro" />                   <!--wheel properties and links definitions-->
@@ -15,4 +19,5 @@
     <xacro:include filename="$(find qupa_description)/urdf/gazebo_plugins.xacro" />                 <!--Gazebo plugins definitions-->
     <xacro:include filename="$(find qupa_description)/urdf/sensors/color.xacro" />
+    <xacro:include filename="$(find qupa_description)/urdf/sensors/led.xacro" />
     <xacro:include filename="$(find qupa_description)/urdf/wheels/caster.xacro" />
     <material name="dark">
@@ -106,28 +111,31 @@
     <xacro:ir_sensor link_name="ir_0"
         joint_name="ir_0_joint"
-        joint_origin_xyz="0.004 -0.056 0.034"
+        joint_origin_xyz="${0.004*ir_inset_scale} ${-0.056*ir_inset_scale} 0.034"
         joint_origin_rpy="${M_PI/2} 0 0" />
     <xacro:ir_sensor link_name="ir_45"
         joint_name="ir_45_joint"
-        joint_origin_xyz="0.04159 -0.0376 0.034"
+        joint_origin_xyz="${0.04159*ir_inset_scale} ${-0.0376*ir_inset_scale} 0.034"
         joint_origin_rpy="${M_PI/2} 0 ${M_PI/4}" />
     <xacro:ir_sensor link_name="ir_90"
         joint_name="ir_90_joint"
-        joint_origin_xyz="0.056 0 0.034"
+        joint_origin_xyz="${0.056*ir_inset_scale} 0 0.034"
         joint_origin_rpy="${M_PI/2} 0 ${M_PI/2}" />
     <xacro:ir_sensor link_name="ir_135"
         joint_name="ir_135_joint"
-        joint_origin_xyz="0.04159 0.0376 0.034"
+        joint_origin_xyz="${0.04159*ir_inset_scale} ${0.0376*ir_inset_scale} 0.034"
         joint_origin_rpy="${M_PI/2} 0 ${3*M_PI/4}" />
     <xacro:ir_sensor link_name="ir_180"
         joint_name="ir_180_joint"
-        joint_origin_xyz="0.004 0.056 0.034"
+        joint_origin_xyz="${0.004*ir_inset_scale} ${0.056*ir_inset_scale} 0.034"
         joint_origin_rpy="${M_PI/2} 0 ${M_PI}" />
     <xacro:ir_sensor link_name="ir_270"
         joint_name="ir_270_joint"
-        joint_origin_xyz="-0.056 0 0.034"
+        joint_origin_xyz="${-0.056*ir_inset_scale} 0 0.034"
         joint_origin_rpy="${M_PI/2} 0 ${-M_PI/2}" />
+    <!-- Floor colour sensor — always present regardless of camera mode -->
+    <xacro:color_camera/>
+    <!-- LED ring — 5 point lights on the dome -->
+    <xacro:led_ring/>
     <xacro:if value="${high_res}">
-        <!-- <xacro:color_camera/> -->
         <xacro:real_cam/>
     </xacro:if>

File: qupa_description/urdf/qupa_real.xacro (robot description, xacro)
@@ -2,7 +2,9 @@
 <!-- Wrapper for the real robot (no module, no high_res camera) -->
 <robot xmlns:xacro="http://www.ros.org/wiki/xacro" name="qupa">
-  <xacro:arg name="tf_prefix" default="qupa"/>
-  <xacro:arg name="high_res"  default="false"/>
-  <xacro:arg name="module"    default="false"/>
+  <xacro:arg name="tf_prefix"        default="qupa"/>
+  <xacro:arg name="high_res"         default="false"/>
+  <xacro:arg name="module"           default="false"/>
+  <!-- Set to true only when spawning in Gazebo (loads gz-harmonic plugins) -->
+  <xacro:arg name="use_sim_plugins"  default="false"/>
   <xacro:include filename="$(find qupa_description)/urdf/qupa.xacro"/>
 </robot>

File: qupa_description/urdf/sensors/color.xacro (robot description, xacro)
@@ -1,84 +1,68 @@
 <?xml version="1.0"?>
 <robot xmlns:xacro="http://www.ros.org/wiki/xacro" name="$(arg tf_prefix)">
+  <!--
+    color.xacro — Downward-facing floor colour sensor.
+    Physical sensor: TCS34725 (I2C) on the real robot.
+    Simulation:      32×32 camera pointing down at 5 Hz (sensor rate).
+                     Colour classification is done by floor_sensor_sim_node at 1 Hz.
+  -->
   <xacro:macro name="color_camera">
     <link name="$(arg tf_prefix)/color_camera_link">
-      <!-- <inertial>
-        <origin
-          xyz="-5.7803E-05 0.0048279 -9.8775E-07"
-          rpy="0 0 0" />
-        <mass
-          value="0.0034683" />
-        <inertia
-          ixx="2.4565E-07"
-          ixy="9.4669E-10"
-          ixz="-3.3359E-11"
-          iyy="4.031E-07"
-          iyz="-7.7399E-12"
-          izz="2.2473E-07" />
-      </inertial> -->
-      <!-- <visual>
-        <origin
-          xyz="0 0 0"
-          rpy="0 0 0" />
-        <geometry>
-          <mesh
-            filename="package://qupa_description/meshes/color.dae" scale="0.6 0.5 0.6"/>
-        </geometry>
-        <material
-          name="">
-          <color
-            rgba="0.79216 0.81961 0.93333 1" />
-        </material>
-      </visual> -->
-      <!-- <collision>
-        <origin
-          xyz="0 0 0"
-          rpy="0 0 0" />
-        <geometry>
-          <mesh
-            filename="package://qupa_description/meshes/color.dae" scale="0.4 0.5 0.4" />
-        </geometry>
-      </collision> -->
+      <!-- Intentionally massless / collision-less — visual sensor only -->
     </link>
     <joint name="color_camera_joint" type="fixed">
-      <origin
-        xyz="-0.043 0 0.009"
-        rpy="0 0 0" />
-      <parent
-        link="$(arg tf_prefix)/base_link" />
-      <child
-        link="$(arg tf_prefix)/color_camera_link" />
-      <axis
-        xyz="0 0 1" />
+      <origin xyz="-0.043 0 0.009" rpy="0 0 0" />
+      <parent link="$(arg tf_prefix)/base_link" />
+      <child  link="$(arg tf_prefix)/color_camera_link" />
+      <axis   xyz="0 0 1" />
     </joint>
-    <gazebo reference="color_camera_link">
-      <sensor  name="$(arg tf_prefix)_color_camera" type="camera">
-        <pose>0 0 0.0 0 0 0</pose>            <!--Ajusta la posición/orientación si es necesario -->
-        <update_rate>30.0</update_rate>           <!-- Frecuencia de actualización en Hz -->
-        <camera>
-          <vertical_fov>1.0</vertical_fov>  <!-- Campo de visión horizontal en radianes -->
-          <image>
-            <width>540</width>                    <!-- Resolución horizontal -->
-            <height>540</height>                  <!-- Resolución vertical -->
-            <format>R8G8B8</format>               <!-- Formato de imagen -->
-          </image>
-          <clip>
-            <near>0.01</near>                     <!-- Distancia mínima del plano de visión -->
-            <far>0.04</far>                        <!-- Distancia máxima del plano de visión -->
-          </clip>
-        </camera>
-        <plugin name="$(arg tf_prefix)_color_sensor" filename="libgazebo_ros_camera.so">
-          <ros>
-            <namespace>$(arg tf_prefix)</namespace>
-          </ros>
-          <alwaysOn>true</alwaysOn>
-          <updateRate>20.0</updateRate>
-          <cameraName>color_camera</cameraName>
-          <imageTopicName>/$(arg tf_prefix)/color_camera/image_raw</imageTopicName>
-          <cameraInfoTopicName>/$(arg tf_prefix)/color_camera/camera_info</cameraInfoTopicName>
-          <frameName>$(arg tf_prefix)/color_camera_link</frameName>
-        </plugin>
-      </sensor>
-    </gazebo>
+    <!-- Gazebo Harmonic: downward-facing camera + LED light (simulation only) -->
+    <xacro:if value="${use_sim_plugins}">
+      <gazebo reference="$(arg tf_prefix)/color_camera_link">
+        <!--
+          Simulated LED — replicates the TCS34725 integrated white LED.
+          A small point light attached to the sensor link guarantees
+          consistent, shadow-free illumination of the floor patch directly
+          below the robot, independent of world lighting and robot body shadows.
+          This also makes the sensor compatible with textured floor materials.
+        -->
+        <light name="$(arg tf_prefix)_floor_led" type="point">
+          <pose>0 0 0 0 0 0</pose>
+          <diffuse>1.0 1.0 1.0 1</diffuse>     <!-- white, neutral -->
+          <specular>0.0 0.0 0.0 1</specular>    <!-- no specular — avoid reflections -->
+          <attenuation>
+            <range>0.12</range>       <!-- 12 cm — only illuminates the floor patch -->
+            <constant>0.8</constant>
+            <linear>0.2</linear>
+            <quadratic>0.05</quadratic>
+          </attenuation>
+          <cast_shadows>false</cast_shadows>    <!-- no shadows from such a close light -->
+        </light>
+        <!--
+          Camera sensor — looks straight down (-Z world).
+          In Gazebo Harmonic the camera looks along its local +X axis.
+          Pitch +π/2 rotates +X → -Z (downward).
+        -->
+        <sensor name="$(arg tf_prefix)_floor_camera" type="camera">
+          <pose>0 0 0 0 1.5708 0</pose>
+          <camera>
+            <horizontal_fov>1.0</horizontal_fov>
+            <image>
+              <width>32</width>
+              <height>32</height>
+              <format>R8G8B8</format>
+            </image>
+            <clip>
+              <near>0.005</near>
+              <far>0.15</far>   <!-- SDF minimum is 0.10 m; 0.15 m clears the floor comfortably -->
+            </clip>
+          </camera>
+          <always_on>true</always_on>
+          <update_rate>5</update_rate>
+          <topic>/$(arg tf_prefix)/floor_camera/image_raw</topic>
+          <gz_frame_id>$(arg tf_prefix)/color_camera_link</gz_frame_id>
+        </sensor>
+      </gazebo>
+    </xacro:if>
   </xacro:macro>
 </robot>
