Commit message: add urdf descriptions for leds sim plugin and stl meshes

File: qupa_description/urdf/sensors/infrared.xacro (robot description, xacro)
@@ -1,10 +1,14 @@
 <?xml version="1.0"?>
 <robot xmlns:xacro="http://www.ros.org/wiki/xacro" name="$(arg tf_prefix)">
-  <!--Xacro Properties-->
-  <xacro:property name="ray_visualizer" value="false" /> <!--Visualize IR sensor in Gazebo-->
-  <!-- IR sensor visual-->
+  <!-- ─────────────────────────────────────────────────────────────────
+       IR SENSOR XACRO  —  QUPA robot
+       Visual meshes for the 6 physical IR sensors (ir_0 … ir_270).
+       The actual range measurement is done by a single GPU-lidar sensor
+       placed at infrared_link that sweeps 360° in 8 samples (45° apart),
+       replicating the real hardware's 8-slot LaserScan output.
+  ───────────────────────────────────────────────────────────────────── -->
+  <!-- Individual IR sensor visual (one per physical sensor position) -->
   <xacro:macro name="ir_sensor" params="link_name joint_name
                                         joint_origin_xyz joint_origin_rpy">
-    <!--Link Definition -->
     <link name="$(arg tf_prefix)/${link_name}">
       <inertial>
@@ -22,5 +26,4 @@
       </visual>
     </link>
-    <!-- Joint Definition -->
     <joint name="${joint_name}" type="fixed">
       <origin xyz="${joint_origin_xyz}" rpy="${joint_origin_rpy}" />
@@ -30,7 +33,15 @@
     </joint>
   </xacro:macro>
-  <!-- IR sensor Macro-->
+  <!-- ─────────────────────────────────────────────────────────────────
+       INFRARED MACRO  —  single sensing link + Gazebo Harmonic sensor
+       Placed at the geometric centre of the IR ring (z=0.034 m above
+       base_link). The GPU-lidar scans 360° in 8 equal steps (45°),
+       matching the real hardware's 8-slot LaserScan convention:
+         slot 0 → 0°    (E)      slot 1 → 45°   (NE)
+         slot 2 → 90°   (N)      slot 3 → 135°  (NW)   [no physical sensor → inf]
+         slot 4 → 180°  (W)      slot 5 → 225°  (SW)   [no physical sensor → inf]
+         slot 6 → 270°  (S)      slot 7 → 315°  (SE)
+  ───────────────────────────────────────────────────────────────────── -->
   <xacro:macro name="infrared" params="joint_origin_xyz joint_origin_rpy">
-    <!--Link Definition -->
     <link name="$(arg tf_prefix)/infrared_link">
       <inertial>
@@ -39,18 +50,11 @@
       </inertial>
       <visual>
-        <geometry>
-          <box size="0.01 0.01 0.01"/>
-        </geometry>
-        <material name="gray">
-          <color rgba="0.5 0.5 0.5 1"/>
-        </material>
+        <geometry><box size="0.01 0.01 0.01"/></geometry>
+        <material name="gray"><color rgba="0.5 0.5 0.5 1"/></material>
       </visual>
       <collision>
-        <geometry>
-          <box size="0.01 0.01 0.01"/>
-        </geometry>
+        <geometry><box size="0.01 0.01 0.01"/></geometry>
       </collision>
     </link>
-    <!-- Joint Definition -->
     <joint name="infrared_joint" type="fixed">
       <origin xyz="${joint_origin_xyz}" rpy="${joint_origin_rpy}" />
@@ -59,36 +63,49 @@
       <axis xyz="0 0 0" />
     </joint>
-    <!-- Gazebo reference and Sensor configuration -->
-    <gazebo reference="infrared_link">
-      <sensor type="ray" name="$(arg tf_prefix)_infrared_sensor">
-        <pose>0 0 0 1.5708 0 0</pose>
-        <visualize>${ray_visualizer}</visualize>
-        <update_rate>30</update_rate>
-        <ray>
-          <scan>
-            <horizontal>
-              <samples>9</samples>
-              <resolution>1</resolution>
-              <min_angle>0</min_angle>
-              <max_angle>${2*M_PI}</max_angle>
-            </horizontal>
-          </scan>
-          <range>
-            <min>0.08</min>
-            <max>0.56</max>
-            <resolution>0.01</resolution>
-          </range>
-          <noise>
-            <type>gaussian</type>
-            <mean>0.0</mean>
-            <stddev>0.005</stddev>
-          </noise>
-        </ray>
-        <plugin name="$(arg tf_prefix)/infrared_plugin" filename="libgazebo_ros_laser.so">
-          <topicName>$(arg tf_prefix)/scan</topicName>
-          <frameName>$(arg tf_prefix)/infrared_link</frameName>
-        </plugin>
-      </sensor>
-    </gazebo>
+    <!-- Gazebo Harmonic: GPU-lidar sensor (gz::sim::systems::Sensors required in world) -->
+    <xacro:if value="${use_sim_plugins}">
+      <gazebo reference="$(arg tf_prefix)/infrared_link">
+        <sensor name="$(arg tf_prefix)_infrared" type="gpu_lidar">
+          <!--
+            Pose inside the sensor rotates the scan plane so that rays are
+            horizontal (parallel to XY of base_link), matching real hardware.
+          -->
+          <pose>0 0 0 1.5708 0 0</pose>
+          <!-- gz-transport topic (bridged to ROS by ros_gz_bridge) -->
+          <topic>/$(arg tf_prefix)/scan</topic>
+          <update_rate>10</update_rate>
+          <gz_frame_id>$(arg tf_prefix)/infrared_link</gz_frame_id>
+          <lidar>
+            <scan>
+              <horizontal>
+                <!--
+                  8 samples over [0, 2π) → rays at 0°, 45°, 90°, 135°,
+                  180°, 225°, 270°, 315° — identical to real LaserScan layout.
+                  Slots 3 (135°) and 5 (225°) have no physical sensor; the
+                  hardware node publishes inf there. Gazebo will publish the
+                  real simulated range for all 8 slots.
+                -->
+                <samples>9</samples>
+                <resolution>1</resolution>
+                <min_angle>0</min_angle>
+                <max_angle>6.28318530718</max_angle>
+              </horizontal>
+            </scan>
+            <range>
+              <min>0.08</min>   <!-- 12 cm — clears robot body (~6 cm radius) -->
+              <max>0.50</max>   <!-- 50 cm -->
+              <resolution>0.01</resolution>
+            </range>
+            <noise>
+              <type>gaussian</type>
+              <mean>0.0</mean>
+              <stddev>0.005</stddev>
+            </noise>
+          </lidar>
+          <always_on>true</always_on>
+          <visualize>true</visualize>
+        </sensor>
+      </gazebo>
+    </xacro:if>
   </xacro:macro>
 </robot>

File: qupa_description/urdf/sensors/mirror.xacro (robot description, xacro)
@@ -1,37 +1,24 @@
 <?xml version="1.0"?>
 <robot xmlns:xacro="http://www.ros.org/wiki/xacro" name="$(arg tf_prefix)">
-    <!-- Properties -->
-    <!-- <xacro:arg name="tf_prefix" default="qupa" /> -->
     <xacro:property name="camera_height" value="0.20" />
-    <!-- Mirror Macro -->
+    <!-- ─────────────────────────────────────────────────────────────────
+         MIRROR — physical mesh (always present, no sensor)
+    ───────────────────────────────────────────────────────────────────── -->
     <xacro:macro name="mirror">
         <link name="$(arg tf_prefix)/mirror_link">
             <inertial>
-            <origin
-                xyz="0 0.0072703 1.0408E-17"
-                rpy="0 0 0" />
-            <mass
-                value="0.00099484" />
-            <inertia
-                ixx="5.9879E-08"
-                ixy="4.6719E-24"
-                ixz="2.2618E-23"
-                iyy="1.0131E-07"
-                iyz="-1.9251E-23"
-                izz="5.9879E-08" />
+                <origin xyz="0 0.0072703 1.0408E-17" rpy="0 0 0" />
+                <mass value="0.00099484" />
+                <inertia ixx="5.9879E-08" ixy="4.6719E-24" ixz="2.2618E-23"
+                         iyy="1.0131E-07" iyz="-1.9251E-23" izz="5.9879E-08" />
             </inertial>
             <visual>
-            <origin
-                xyz="0 0 0"
-                rpy="0 0 0" />
-            <geometry>
-                <mesh
-                filename="package://qupa_description/meshes/mirror.stl" />
-            </geometry>
-            <material
-                name="">
-                <color
-                rgba="0.74902 0.74902 0.74902 1" />
-            </material>
+                <origin xyz="0 0 0" rpy="0 0 0" />
+                <geometry>
+                    <mesh filename="package://qupa_description/meshes/mirror.stl" />
+                </geometry>
+                <material name="">
+                    <color rgba="0.74902 0.74902 0.74902 1" />
+                </material>
             </visual>
         </link>
@@ -43,103 +30,124 @@
         </joint>
     </xacro:macro>
-    <!-- Logical Camera Macro -->
+    <!-- ─────────────────────────────────────────────────────────────────
+         LOGICAL CAMERA  (high_res:=false)
+         Cone-shaped sensor from the mirror point of reference.
+         Simulates the conical FOV that the hyperbolic mirror provides.
+         No rendering required — works without GPU.
+    ───────────────────────────────────────────────────────────────────── -->
     <xacro:macro name="log_cam">
-        <!--Logical Camera Frame-->
         <link name="$(arg tf_prefix)/logical_camera_link">
             <inertial>
                 <mass value="0.001" />
                 <origin xyz="0 0 0" rpy="0 0 0" />
-                <inertia ixx="1.875e-8" ixy="0.0" ixz="0.0" iyy="1.875e-8" iyz="0.0" izz="1.25e-8" />
+                <inertia ixx="1.875e-8" ixy="0.0" ixz="0.0"
+                         iyy="1.875e-8" iyz="0.0" izz="1.25e-8" />
             </inertial>
             <collision>
                 <origin xyz="0 0 0" rpy="0 0 0" />
-                <geometry>
-                    <cylinder radius="0.005" length="0.01" />
-                </geometry>
+                <geometry><cylinder radius="0.005" length="0.01"/></geometry>
             </collision>
         </link>
-        <!--Logical Camera joint-->
         <joint name="logical_camera_joint" type="fixed">
             <parent link="$(arg tf_prefix)/base_link" />
             <child link="$(arg tf_prefix)/logical_camera_link" />
-            <origin xyz="0 0 ${camera_height}"  rpy="0 1.5708 0" />
+            <origin xyz="0 0 ${camera_height}" rpy="0 1.5708 0" />
         </joint>
-        <!--Logical Camera PLugin-->
-        <gazebo reference="logical_camera_link">
-            <sensor name="$(arg tf_prefix)_mirror" type="logical_camera">
-                <logical_camera>
-                    <near>0.04</near>
-                    <far>0.20</far>
-                    <horizontal_fov>2.5</horizontal_fov>
-                    <aspect_ratio>${240.0/240.0}</aspect_ratio>
-                </logical_camera>
-                <visualize>false</visualize>
-                <always_on>true</always_on>
-                <update_rate>20</update_rate>
-            </sensor>
-        </gazebo>
+        <!-- Gazebo Harmonic: logical_camera sensor (no rendering, no GPU needed) -->
+        <xacro:if value="${use_sim_plugins}">
+            <gazebo reference="$(arg tf_prefix)/logical_camera_link">
+                <sensor name="$(arg tf_prefix)_mirror" type="logical_camera">
+                    <logical_camera>
+                        <near>0.04</near>
+                        <far>0.20</far>
+                        <horizontal_fov>2.5</horizontal_fov>
+                        <aspect_ratio>1.0</aspect_ratio>
+                    </logical_camera>
+                    <visualize>false</visualize>
+                    <always_on>true</always_on>
+                    <update_rate>20</update_rate>
+                    <topic>/$(arg tf_prefix)/logical_camera</topic>
+                </sensor>
+            </gazebo>
+        </xacro:if>
     </xacro:macro>
+    <!-- ─────────────────────────────────────────────────────────────────
+         FISHEYE CAMERA  (high_res:=true)
+         Wide-angle camera that replicates the hyperbolic mirror + camera
+         setup of the real robot. Uses Gazebo Harmonic's wideanglecamera
+         sensor with a custom lens function (tan projection, 360° FOV).
+         Requires: gz-sim-sensors-system with ogre2 render engine.
+         The raw image is published on gz-transport only — no ROS image
+         topic is created. The camera_sim_node reads it via gz-transport
+         Python and publishes only camera/detections (DetectionArray).
+    ───────────────────────────────────────────────────────────────────── -->
     <xacro:macro name="real_cam">
-        <!--Logical Camera Frame-->
         <link name="$(arg tf_prefix)/camera_link">
             <inertial>
                 <mass value="0.001" />
                 <origin xyz="0 0 0" rpy="0 0 0" />
-                <inertia ixx="1.875e-8" ixy="0.0" ixz="0.0" iyy="1.875e-8" iyz="0.0" izz="1.25e-8" />
+                <inertia ixx="1.875e-8" ixy="0.0" ixz="0.0"
+                         iyy="1.875e-8" iyz="0.0" izz="1.25e-8" />
             </inertial>
             <collision>
                 <origin xyz="0 0 0" rpy="0 0 0" />
-                <geometry>
-                    <cylinder radius="0.005" length="0.01" />
-                </geometry>
+                <geometry><cylinder radius="0.005" length="0.01"/></geometry>
             </collision>
         </link>
-        <!--Logical Camera joint-->
+        <!--
+            Joint at camera_height (0.20 m) pointing upward toward the mirror.
+            rpy="0 1.5708 0" rotates the link so the camera faces the mirror.
+        -->
         <joint name="camera_joint" type="fixed">
             <parent link="$(arg tf_prefix)/base_link" />
             <child link="$(arg tf_prefix)/camera_link" />
-            <origin xyz="0 0 ${camera_height}"  rpy="0 1.5708 0" />
+            <origin xyz="0 0 ${camera_height}" rpy="0 1.5708 0" />
         </joint>
-        <gazebo reference="camera_link">
-            <sensor name="$(arg tf_prefix)_camera"  type="wideanglecamera">
-                <camera>
-                    <horizontal_fov>6.283</horizontal_fov><!-- 6.28 for 360 -->
-                    <image>
-                        <width>720</width>
-                        <height>720</height>
-                    </image>
-                    <clip>
-                        <near>0.1</near>
-                        <far>0.8</far>
-                    </clip>
-                    <lens>                          <!-- A new section named `lens`. -->
-                        <type>custom</type>         <!-- type element is mandatory -->
-                        <custom_function>
-                            <c1>1.05</c1>            <!-- linear scaling default:1.05 -->
-                            <c2>3</c2>              <!-- angle scaling  default:4 -->
-                            <f>1.0</f>              <!-- one more scaling parameter default:1.0-->
-                            <fun>tan</fun>          <!-- one of sin,tan,id default:tan -->
-                        </custom_function>
-                        <!-- if it is set to `true` your horizontal FOV will ramain as defined -->
-                        <!-- othervise it depends on lens type and custom function, if there is one -->
-                        <scale_to_hfov>true</scale_to_hfov>
-                        <!-- clip everything that is outside of this angle -->
-                        <cutoff_angle>2.5</cutoff_angle>
-                        <!-- resolution of the cubemap texture, the highter it is - the sharper is your image -->
-                        <env_texture_size>720</env_texture_size>
-                    </lens>
-                </camera>
-                <always_on>1</always_on>
-                <update_rate>30</update_rate>
-                <plugin name="$(arg tf_prefix)_gazebo_ros_camera" filename="libgazebo_ros_camera.so">
-                    <alwaysOn>true</alwaysOn>
-                    <updateRate>20.0</updateRate>
-                    <cameraName>$(arg tf_prefix)/mirror_camera</cameraName>
-                    <imageTopicName>/$(arg tf_prefix)/camera/image_raw</imageTopicName>
-                    <cameraInfoTopicName>/$(arg tf_prefix)/camera/camera_info</cameraInfoTopicName>
-                    <frameName>$(arg tf_prefix)/camera_link</frameName>
-                </plugin>
-            </sensor>
-        </gazebo>
+        <!-- Gazebo Harmonic: wideanglecamera sensor (requires ogre2 rendering) -->
+        <xacro:if value="${use_sim_plugins}">
+            <gazebo reference="$(arg tf_prefix)/camera_link">
+                <sensor name="$(arg tf_prefix)_camera" type="wideanglecamera">
+                    <camera>
+                        <!-- 360° horizontal FOV — full surround view like the mirror -->
+                        <!-- SDF max is 2π = 6.28318…; 6.2832 exceeds it by rounding -->
+                        <horizontal_fov>6.28318</horizontal_fov>
+                        <image>
+                            <width>720</width>
+                            <height>720</height>
+                            <format>R8G8B8</format>
+                        </image>
+                        <clip>
+                            <near>0.05</near>
+                            <far>5.0</far>
+                        </clip>
+                        <!--
+                            Custom fisheye lens — replicates the tan-projection
+                            that the hyperbolic mirror introduces.
+                            r(θ) = c1 * tan(c2 * θ + f)
+                        -->
+                        <lens>
+                            <type>custom</type>
+                            <custom_function>
+                                <c1>1.05</c1>   <!-- radial scaling -->
+                                <c2>3.0</c2>    <!-- angle scaling  -->
+                                <f>1.0</f>      <!-- offset         -->
+                                <fun>tan</fun>  <!-- projection: tan, sin or id -->
+                            </custom_function>
+                            <!-- Keep horizontal_fov as defined above -->
+                            <scale_to_hfov>true</scale_to_hfov>
+                            <!-- Clip rays beyond this half-angle (≈143°) -->
+                            <cutoff_angle>2.5</cutoff_angle>
+                            <!-- Cubemap resolution — trade-off: quality vs GPU cost -->
+                            <env_texture_size>512</env_texture_size>
+                        </lens>
+                    </camera>
+                    <always_on>true</always_on>
+                    <update_rate>10</update_rate>  <!-- real node runs at 3 Hz; 10 Hz gives margin -->
+                    <!-- gz-transport topic consumed by camera_sim_node via gz-transport Python -->
+                    <topic>/$(arg tf_prefix)/camera/image_raw</topic>
+                    <gz_frame_id>$(arg tf_prefix)/camera_link</gz_frame_id>
+                </sensor>
+            </gazebo>
+        </xacro:if>
     </xacro:macro>
 </robot>

File: qupa_description/urdf/wheels/caster.xacro (robot description, xacro)
@@ -33,12 +33,24 @@
       <child link="${link_name}" />
     </joint>
+    <!-- Gazebo Harmonic: friction inside <collision><surface> (SDF 1.9 format) -->
     <gazebo reference="${link_name}">
-      <mu1>0.1</mu1>
-      <mu2>0.1</mu2>
-      <kp>1000000.0</kp>
-      <kd>100.0</kd>
-      <minDepth>0.001</minDepth>
-      <maxVel>1.0</maxVel>
-      <!-- <material>Gazebo/FlatBlack</material> -->
+      <collision>
+        <surface>
+          <friction>
+            <ode>
+              <mu>0.1</mu>
+              <mu2>0.1</mu2>
+            </ode>
+          </friction>
+          <contact>
+            <ode>
+              <kp>1000000.0</kp>
+              <kd>100.0</kd>
+              <min_depth>0.001</min_depth>
+              <max_vel>1.0</max_vel>
+            </ode>
+          </contact>
+        </surface>
+      </collision>
     </gazebo>
   </xacro:macro>

File: qupa_description/urdf/wheels/wheel.xacro (robot description, xacro)
@@ -59,11 +59,24 @@
       <dynamics damping="${wheel_damping}" friction="${wheel_friction}" />
     </joint>
+    <!-- Gazebo Harmonic: friction inside <collision><surface> (SDF 1.9 format) -->
     <gazebo reference="${wheel_name}">
-      <mu>${wheel_friction_mu}</mu>
-      <mu2>${wheel_friction_mu2}</mu2>
-      <kp>${contact_kp}</kp>
-      <kd>${contact_kd}</kd>
-      <maxVel>${max_contact_vel}</maxVel>
-      <minDepth>${min_contact_depth}</minDepth>
+      <collision>
+        <surface>
+          <friction>
+            <ode>
+              <mu>${wheel_friction_mu}</mu>
+              <mu2>${wheel_friction_mu2}</mu2>
+            </ode>
+          </friction>
+          <contact>
+            <ode>
+              <kp>${contact_kp}</kp>
+              <kd>${contact_kd}</kd>
+              <max_vel>${max_contact_vel}</max_vel>
+              <min_depth>${min_contact_depth}</min_depth>
+            </ode>
+          </contact>
+        </surface>
+      </collision>
     </gazebo>
   </xacro:macro>
