Commit message: update urdf

File: qupa_description/urdf/bases/base.xacro (robot description, xacro)
@@ -5,9 +5,9 @@
     <!-- Real robot is white -->
     <material name="white">
-        <color rgba="0.9 0.9 0.9 1.0" />
+        <color rgba="1.0 1.0 1.0 1.0" />
     </material>
     <!-- Acrylic dome: WHITE translucent diffuser the LEDs glow through.
          acrylic_alpha: 0 = invisible, 1 = fully opaque. Lower = lighter/clearer. -->
-    <xacro:property name="acrylic_alpha" value="0.90" />
+    <xacro:property name="acrylic_alpha" value="0.98" />
     <material name="acrylic">
         <color rgba="1.0 1.0 1.0 ${acrylic_alpha}" />

File: qupa_description/urdf/bases/module.xacro (robot description, xacro)
@@ -2,5 +2,5 @@
 <robot xmlns:xacro="http://www.ros.org/wiki/xacro">
     <xacro:property name="base_mass" value="1" />
-    <xacro:property name="base_scale" value="1 1 1" />
+    <xacro:property name="base_scale" value="0.85 0.85 1" />
     <!--Base with Module installed-->
     <xacro:macro name="module">
@@ -17,18 +17,46 @@
                     izz="0.00180" />
                 </inertial>
-            <visual>
-                <origin xyz="0 0 0" rpy="0 0 0" />
-                <geometry>
-                    <mesh filename="package://qupa_description/meshes/module.dae" scale="${base_scale}" />
-                </geometry>
-            </visual>
-            <collision>
-                <origin xyz="0 0 0" rpy="0 0 0" />
-                <geometry>
-                    <mesh filename="package://qupa_description/meshes/module.dae" scale="${base_scale}" />
+            <!-- base_w_module.stl: base sin domo, con soporte del módulo -->
+            <visual>
+                <origin xyz="0 0 0" rpy="0 0 0" />
+                <geometry>
+                    <mesh filename="package://qupa_description/meshes/base_w_module.stl" scale="${base_scale}" />
+                </geometry>
+                <material name="white" />
+            </visual>
+            <collision>
+                <origin xyz="0 0 0" rpy="0 0 0" />
+                <geometry>
+                    <mesh filename="package://qupa_description/meshes/base_w_module.stl" scale="${base_scale}" />
                 </geometry>
                 <self_collide>false</self_collide>
             </collision>
         </link>
+        <!-- Domo acrílico — link separado para que led_sim_node pueda cambiar
+             su color emissivo igual que en la config sin módulo. -->
+        <link name="$(arg tf_prefix)/acrylic_dome_link">
+            <inertial>
+                <mass value="1e-5" />
+                <origin xyz="0 0 0" rpy="0 0 0" />
+                <inertia ixx="1e-9" ixy="0" ixz="0"
+                         iyy="1e-9" iyz="0" izz="1e-9" />
+            </inertial>
+            <visual>
+                <origin xyz="0 0 0" rpy="0 0 0" />
+                <geometry>
+                    <mesh filename="package://qupa_description/meshes/dome.stl" scale="${base_scale}" />
+                </geometry>
+                <material name="acrylic" />
+            </visual>
+        </link>
+        <joint name="acrylic_dome_joint" type="fixed">
+            <parent link="$(arg tf_prefix)/base_link" />
+            <child  link="$(arg tf_prefix)/acrylic_dome_link" />
+            <origin xyz="0 0 0.048" rpy="0 0 0" />
+        </joint>
+        <gazebo reference="acrylic_dome_joint">
+            <disableFixedJointLumping>true</disableFixedJointLumping>
+            <preserveFixedJoint>true</preserveFixedJoint>
+        </gazebo>
         <joint name="imu_joint" type="fixed">
             <parent link="$(arg tf_prefix)/base_link"/>
@@ -91,4 +119,5 @@
             <axis xyz="0 0 1"/>
             <limit lower="-3.1416" upper="3.1416" effort="100" velocity="1.0"/>
+            <dynamics damping="0.1" friction="0.0"/>
         </joint>
     </xacro:macro>
@@ -128,9 +157,23 @@
             <child link="Left_Link_2" />
             <axis xyz="0 0 1" />
-            <limit  lower="-3.1416"
-                    upper="3.1416"
-                    effort="10"
-                    velocity="1.0" />
-        </joint>
+            <limit lower="-3.1416" upper="3.1416" effort="10" velocity="1.0" />
+            <dynamics damping="0.1" friction="0.1"/>
+        </joint>
+        <!-- Closure tip: punto de cierre fijo a Left_Link_2.
+             Pose tomada del joint "closure" original del URDF de Gazebo Classic. -->
+        <link name="Left_closure_tip">
+            <inertial>
+                <mass value="0.001"/>
+                <inertia ixx="1e-6" ixy="0" ixz="0" iyy="1e-6" iyz="0" izz="1e-6"/>
+            </inertial>
+        </link>
+        <joint name="Left_closure_tip_joint" type="fixed">
+            <origin xyz="0.09 0 0" rpy="3.1416 0 -0.33145"/>
+            <parent link="Left_Link_2"/>
+            <child link="Left_closure_tip"/>
+        </joint>
+        <gazebo reference="Left_closure_tip_joint">
+            <preserveFixedJoint>true</preserveFixedJoint>
+        </gazebo>
     </xacro:macro>
     <!--Link 3-->
@@ -164,14 +207,28 @@
             </collision>
         </link>
-        <joint name="Right_joint_2"  type="revolute">
+        <joint name="Right_joint_2" type="revolute">
             <origin xyz="${xyz}" rpy="${rpy}" />
             <parent link="Right_Link_1" />
             <child  link="Right_Link_2" />
             <axis   xyz="0 0 1" />
-            <limit
-                lower="-3.1416"
-                upper="3.1416"
-                effort="10"
-                velocity="1.0" />
+            <limit lower="-3.1416" upper="3.1416" effort="10" velocity="1.0" />
+            <dynamics damping="0.1" friction="0.1"/>
+        </joint>
+        <!-- Closure dummy: link en la PUNTA de Right_Link_2 (xyz=0.09 0 0 en frame local).
+             El DetachableJoint suelda Left_closure_tip con este punto, cerrando la cadena.
+             Revolute Z: equivalente al joint "closure" type="revolute" del URDF ROS1. -->
+        <link name="Right_closure_dummy">
+            <inertial>
+                <mass value="0.001"/>
+                <inertia ixx="1e-6" ixy="0" ixz="0" iyy="1e-6" iyz="0" izz="1e-6"/>
+            </inertial>
+        </link>
+        <joint name="Right_closure_joint" type="revolute">
+            <origin xyz="0.09 0 0" rpy="3.1416 0 -0.93631"/>
+            <parent link="Right_Link_2"/>
+            <child link="Right_closure_dummy"/>
+            <axis xyz="0 0 1"/>
+            <limit lower="-3.14" upper="3.14" effort="0" velocity="10"/>
+            <dynamics damping="0.1" friction="0.0"/>
         </joint>
     </xacro:macro>
@@ -229,19 +286,15 @@
                 effort="10"
                 velocity="0.01" />
-        </joint>
-        <!-- Joint pasivo entre Left_Link_2 y closure_link -->
-          <gazebo>
-            <joint name="closure" type="revolute">
-            <parent>Left_Link_2</parent>
-            <child>Right_Link_2</child>
-            <pose>0.09 0 0 3.1416 0 -0.33145</pose>
-            <axis>
-                <xyz>0 0 1</xyz>
-                <limit>
-                <lower>-6.2</lower>
-                <upper>6.2</upper>
-                </limit>
-            </axis>
-            </joint>
+            <dynamics damping="0.1" friction="0.0"/>
+        </joint>
+        <!-- DetachableJoint: suelda Left_closure_tip con Right_closure_dummy,
+             cerrando físicamente la cadena. DART + PGS solver resuelve el loop. -->
+        <gazebo>
+            <plugin filename="libgz-sim-detachable-joint-system.so"
+                    name="gz::sim::systems::DetachableJoint">
+                <parent_link>Left_closure_tip</parent_link>
+                <child_model>$(arg tf_prefix)</child_model>
+                <child_link>Right_closure_dummy</child_link>
+            </plugin>
         </gazebo>
     </xacro:macro>

File: qupa_description/urdf/gazebo_plugins.xacro (robot description, xacro)
@@ -7,4 +7,18 @@
   -->
   <xacro:if value="${use_sim_plugins}">
+    <!-- ───────────────────────────────────────────────────────────────
+         JOINT STATE PUBLISHER  (gz::sim::systems::JointStatePublisher)
+         Publishes wheel joint positions to gz-transport so the
+         ros_gz_bridge can forward them to ROS /joint_states and
+         robot_state_publisher can compute the wheel TF frames.
+    ─────────────────────────────────────────────────────────────────── -->
+    <gazebo>
+      <plugin filename="gz-sim-joint-state-publisher-system"
+              name="gz::sim::systems::JointStatePublisher">
+        <topic>/$(arg tf_prefix)/joint_states</topic>
+        <joint_name>L_wheel_joint</joint_name>
+        <joint_name>R_wheel_joint</joint_name>
+      </plugin>
+    </gazebo>
     <!-- ───────────────────────────────────────────────────────────────
          DIFFERENTIAL DRIVE  (gz::sim::systems::DiffDrive)

File: qupa_description/urdf/qupa.xacro (robot description, xacro)
@@ -33,5 +33,8 @@
     <xacro:if value="${module}">
         <!--Xacro properties changes-->
-        <xacro:property name="base_height" value="0.04" />
+        <xacro:property name="base_height"  value="0.04" />
+        <!-- Module adds ~24 cm of height → camera/mirror sit 44 cm above ground -->
+        <xacro:property name="mirror_height" value="0.24" />
+        <xacro:property name="camera_height" value="0.24" />
         <xacro:module/>               <!--Module Base-->
         <!--Links-->
@@ -53,27 +56,47 @@
             rpy="0 0 0.76626"/>
         <xacro:EE/>
-        <!--Transmissions-->
-        <xacro:transmission_effort  name="trans_motor_left_link_1"
-                                    joint_name="Left_joint_1"
-                                    actuator_name="left_motor"/>
-        <xacro:transmission_effort  name="trans_motor_right_link_1"
-                                    joint_name="Right_joint_1"
-                                    actuator_name="right_motor"/>
-        <xacro:transmission_passive name="left_link_1_left_link_2"
-                                    joint_name="Left_joint_2"
-                                    actuator_name="left_1to2"/>
-        <xacro:transmission_passive name="right_link_1_right_link_2"
-                                    joint_name="Right_joint_2"
-                                    actuator_name="right_1to2"/>
-        <xacro:transmission_effort  name="end_effector_motor"
-                                    joint_name="EE_joint"
-                                    actuator_name="ee_motor"/>
-        <!--plugin-->
-        <gazebo>
-            <plugin name="gazebo_ros_control" filename="libgazebo_ros_control.so">
-                <robotNamespace>$(arg tf_prefix)</robotNamespace>
-                <robotSimType>gazebo_ros_control/ClosedLoopHWSim</robotSimType>
-            </plugin>
-        </gazebo>
+        <!-- ── ros2_control — reemplaza las transmisiones de ROS 1 ──────────
+             Left_joint_2 y Right_joint_2 son PASIVOS: los maneja DART a través
+             del joint "closure" de SDF. Solo se declaran los joints actuados.
+             Requiere: sudo apt install ros-jazzy-gz-ros2-control
+        -->
+        <ros2_control name="$(arg tf_prefix)_arm" type="system">
+            <hardware>
+                <plugin>gz_ros2_control/GazeboSimSystem</plugin>
+            </hardware>
+            <!-- Joints actuados -->
+            <joint name="Left_joint_1">
+                <command_interface name="effort"/>
+                <state_interface name="position"/>
+                <state_interface name="velocity"/>
+            </joint>
+            <joint name="Right_joint_1">
+                <command_interface name="effort"/>
+                <state_interface name="position"/>
+                <state_interface name="velocity"/>
+            </joint>
+            <joint name="EE_joint">
+                <command_interface name="effort"/>
+                <state_interface name="position"/>
+                <state_interface name="velocity"/>
+            </joint>
+            <!-- Left_joint_2 y Right_joint_2 son pasivos — los mueve el DetachableJoint
+                 + física DART. No se declaran en ros2_control. -->
+        </ros2_control>
+        <!-- ── gz_ros2_control plugin (Gazebo Harmonic) ──────────────────
+             Reemplaza libgazebo_ros_control.so / ClosedLoopHWSim de ROS 1.
+             La cadena cerrada (joint "closure") la resuelve DART nativamente.
+        -->
+        <xacro:if value="${use_sim_plugins}">
+            <gazebo>
+                <plugin filename="gz_ros2_control-system"
+                        name="gz_ros2_control::GazeboSimROS2ControlPlugin">
+                    <parameters>$(find qupa_simulation)/config/module_controllers.yaml</parameters>
+                    <ros>
+                        <namespace>$(arg tf_prefix)</namespace>
+                    </ros>
+                </plugin>
+            </gazebo>
+        </xacro:if>
     </xacro:if>
     <xacro:unless value="${module}">

File: qupa_description/urdf/sensors/color.xacro (robot description, xacro)
@@ -49,11 +49,11 @@
             <horizontal_fov>1.0</horizontal_fov>
             <image>
-              <width>32</width>
-              <height>32</height>
+              <width>4</width>
+              <height>4</height>
               <format>R8G8B8</format>
             </image>
             <clip>
               <near>0.005</near>
-              <far>0.15</far>   <!-- SDF minimum is 0.10 m; 0.15 m clears the floor comfortably -->
+              <far>0.15</far>
             </clip>
           </camera>
@@ -61,5 +61,4 @@
           <update_rate>5</update_rate>
           <topic>/$(arg tf_prefix)/floor_camera/image_raw</topic>
-          <gz_frame_id>$(arg tf_prefix)/color_camera_link</gz_frame_id>
         </sensor>
       </gazebo>

File: qupa_description/urdf/sensors/mirror.xacro (robot description, xacro)
@@ -1,5 +1,5 @@
 <?xml version="1.0"?>
 <robot xmlns:xacro="http://www.ros.org/wiki/xacro" name="$(arg tf_prefix)">
-    <xacro:property name="camera_height" value="0.20" />
+    <xacro:property name="camera_height" value="0.18" />
     <!-- ─────────────────────────────────────────────────────────────────
          MIRROR — physical mesh (always present, no sensor)
@@ -113,6 +113,6 @@
                         <horizontal_fov>6.28318</horizontal_fov>
                         <image>
-                            <width>720</width>
-                            <height>720</height>
+                            <width>640</width>
+                            <height>480</height>
                             <format>R8G8B8</format>
                         </image>
@@ -129,22 +129,33 @@
                             <type>custom</type>
                             <custom_function>
-                                <c1>1.05</c1>   <!-- radial scaling -->
-                                <c2>3.0</c2>    <!-- angle scaling  -->
-                                <f>1.0</f>      <!-- offset         -->
-                                <fun>tan</fun>  <!-- projection: tan, sin or id -->
+                                <!--
+                                    FÓRMULA REAL del shader (wide_lens_map_fp.glsl):
+                                      r = c1 * f * fun(theta / c2)
+                                    c2 DIVIDE theta (no multiplica).
+                                    Con scale_to_hfov=true y hfov=360°, Gazebo ignora c1 y f
+                                    y calcula f_eff = 1/fun(180°/c2).
+                                    Con fun=sin, c2=2:
+                                      f_eff = 1/sin(90°) = 1.0  →  sin monótona en [0°,180°] ✓
+                                      θ=  0° → r = 0.000  (centro)
+                                      θ= 90° → r = sin(45°) = 0.707  (horizonte al 70.7 %)
+                                      θ=101° → r = sin(50.5°) = 0.771  (corte al 77.1 %)
+                                      θ=180° → r = 1.000  (punto de normalización)
+                                    | anterior: c1=1.05 c2=3.0 f=1.0 fun=tan cutoff=2.5
+                                -->
+                                <c1>1.0</c1>
+                                <c2>2.0</c2>    <!-- theta/c2=theta/2: sin monótona hasta 180° -->
+                                <f>1.0</f>      <!-- ignorado por scale_to_hfov=true -->
+                                <fun>sin</fun>
                             </custom_function>
-                            <!-- Keep horizontal_fov as defined above -->
                             <scale_to_hfov>true</scale_to_hfov>
-                            <!-- Clip rays beyond this half-angle (≈143°) -->
-                            <cutoff_angle>2.5</cutoff_angle>
-                            <!-- Cubemap resolution — trade-off: quality vs GPU cost -->
+                            <!-- cutoff = 101° = φ_max del espejo real | anterior: 2.5 rad -->
+                            <cutoff_angle>1.763</cutoff_angle>
                             <env_texture_size>512</env_texture_size>
                         </lens>
                     </camera>
                     <always_on>true</always_on>
-                    <update_rate>10</update_rate>  <!-- real node runs at 3 Hz; 10 Hz gives margin -->
+                    <update_rate>5</update_rate>  <!-- real node runs at 3 Hz; 10 Hz gives margin -->
                     <!-- gz-transport topic consumed by camera_sim_node via gz-transport Python -->
                     <topic>/$(arg tf_prefix)/camera/image_raw</topic>
-                    <gz_frame_id>$(arg tf_prefix)/camera_link</gz_frame_id>
                 </sensor>
             </gazebo>
